File: SusPad-PCB/SusPad-PCB.kicad_pcb (KiCad board)
At the start: 2 copper layers, 189 x 106 mm, 33 parts

Commit message: updated pcb
Parts:
- removed the REF** at (138.5, 116.2)
- removed the REF** at (216.5, 116.2)
Routing:
- net (no net): track 2580.6 -> 2565.2 mm, vias 40 -> 38
Other:
- board size 189 x 106 mm -> 87 x 106 mm
- board text added: "DEBUG"
- board text added: "Design by Ben The Builder"
